Commit message: fix edmo xacro model

File: src/edmo_snake_description/urdf/edmo_snake_backup.xacro (robot description, xacro)
@@ -4,10 +4,4 @@
 <xacro:include filename="$(find edmo_snake_description)/urdf/edmo_snake.trans" />
 <xacro:include filename="$(find edmo_snake_description)/urdf/edmo_snake.gazebo" />
-<xacro:property name="base_y_offset" value="0.02" />
-<xacro:property name="arm_x_offset" value="0.027" />
-<xacro:property name="arm_z_offset" value="0.02" />
-<xacro:property name="cover_z_offset" value="0.02" />
-<xacro:property name="straight_connector_x_offset" value="0.06" />
-<xacro:property name="second_arm_x_offset" value="0.16" />
 <link name="dummy">
 </link>
@@ -39,5 +33,5 @@
   </inertial>
   <visual>
-    <origin xyz="-${arm_x_offset} -0.0 -${arm_z_offset}" rpy="0 0 0"/>
+    <origin xyz="-0.038414 -0.041832 0.002983" rpy="0 0 0"/>
     <geometry>
       <mesh filename="package://edmo_snake_description/meshes/arm_1_1.stl" scale="0.001 0.001 0.001"/>
@@ -46,5 +40,5 @@
   </visual>
   <collision>
-    <origin xyz="-${arm_x_offset} -0.0 -${arm_z_offset}" rpy="0 0 0"/>
+    <origin xyz="-0.038414 -0.041832 0.002983" rpy="0 0 0"/>
     <geometry>
       <mesh filename="package://edmo_snake_description/meshes/arm_1_1.stl" scale="0.001 0.001 0.001"/>
@@ -59,5 +53,5 @@
   </inertial>
   <visual>
-    <origin xyz="-0.0 0.0 -${cover_z_offset}" rpy="0 0 0"/>
+    <origin xyz="-0.043315 0.003782 -0.02005" rpy="0 0 0"/>
     <geometry>
       <mesh filename="package://edmo_snake_description/meshes/cover_1_1.stl" scale="0.001 0.001 0.001"/>
@@ -66,5 +60,5 @@
   </visual>
   <collision>
-    <origin xyz="-0.0 0.0 -${cover_z_offset}" rpy="0 0 0"/>
+    <origin xyz="-0.043315 0.003782 -0.02005" rpy="0 0 0"/>
     <geometry>
       <mesh filename="package://edmo_snake_description/meshes/cover_1_1.stl" scale="0.001 0.001 0.001"/>
@@ -79,5 +73,5 @@
   </inertial>
   <visual>
-    <origin xyz="0.0 0.0 0.0" rpy="0 0 0"/>
+    <origin xyz="-0.089365 -0.014468 -0.0201" rpy="0 0 0"/>
     <geometry>
       <mesh filename="package://edmo_snake_description/meshes/straight_connector_1_1.stl" scale="0.001 0.001 0.001"/>
@@ -86,5 +80,5 @@
   </visual>
   <collision>
-    <origin xyz="0.0 0.0 0.0" rpy="0 0 0"/>
+    <origin xyz="-0.089365 -0.014468 -0.0201" rpy="0 0 0"/>
     <geometry>
       <mesh filename="package://edmo_snake_description/meshes/straight_connector_1_1.stl" scale="0.001 0.001 0.001"/>
@@ -99,5 +93,5 @@
   </inertial>
   <visual>
-    <origin xyz="-0.0 -0.0 -0.0" rpy="0 0 0"/>
+    <origin xyz="-0.094365 -0.014468 -0.0201" rpy="0 0 0"/>
     <geometry>
       <mesh filename="package://edmo_snake_description/meshes/base_2_1.stl" scale="0.001 0.001 0.001"/>
@@ -106,5 +100,5 @@
   </visual>
   <collision>
-    <origin xyz="-0.0 -0.0 -0.0" rpy="0 0 0"/>
+    <origin xyz="-0.094365 -0.014468 -0.0201" rpy="0 0 0"/>
     <geometry>
       <mesh filename="package://edmo_snake_description/meshes/base_2_1.stl" scale="0.001 0.001 0.001"/>
@@ -119,5 +113,5 @@
   </inertial>
   <visual>
-    <origin xyz="-0.0 0.0 -0.0" rpy="0 0 0"/>
+    <origin xyz="-0.176165 0.003782 -0.0201" rpy="0 0 0"/>
     <geometry>
       <mesh filename="package://edmo_snake_description/meshes/cover_2_1.stl" scale="0.001 0.001 0.001"/>
@@ -126,5 +120,5 @@
   </visual>
   <collision>
-    <origin xyz="-0.0 0.0 -0.0" rpy="0 0 0"/>
+    <origin xyz="-0.176165 0.003782 -0.0201" rpy="0 0 0"/>
     <geometry>
       <mesh filename="package://edmo_snake_description/meshes/cover_2_1.stl" scale="0.001 0.001 0.001"/>
@@ -139,14 +133,14 @@
   </inertial>
   <visual>
-    <origin xyz="-${arm_x_offset} -0.0 -${arm_z_offset}" rpy="0 0 0"/>
-    <geometry>
-      <mesh filename="package://edmo_snake_description/meshes/arm_1_1.stl" scale="0.001 0.001 0.001"/>
-    </geometry>
-    <material name="silver"/>
-  </visual>
-  <collision>
-    <origin xyz="-${arm_x_offset} -0.0 -${arm_z_offset}" rpy="0 0 0"/>
-    <geometry>
-      <mesh filename="package://edmo_snake_description/meshes/arm_1_1.stl" scale="0.001 0.001 0.001"/>
+    <origin xyz="-0.171314 -0.174682 0.002933" rpy="0 0 0"/>
+    <geometry>
+      <mesh filename="package://edmo_snake_description/meshes/arm_2_1.stl" scale="0.001 0.001 0.001"/>
+    </geometry>
+    <material name="silver"/>
+  </visual>
+  <collision>
+    <origin xyz="-0.171314 -0.174682 0.002933" rpy="0 0 0"/>
+    <geometry>
+      <mesh filename="package://edmo_snake_description/meshes/arm_2_1.stl" scale="0.001 0.001 0.001"/>
     </geometry>
   </collision>
@@ -159,5 +153,5 @@
   </inertial>
   <visual>
-    <origin xyz="-${second_arm_x_offset} -0.0 -${arm_z_offset}" rpy="0 0 0"/>
+    <origin xyz="-0.222215 -0.014468 -0.02015" rpy="0 0 0"/>
     <geometry>
       <mesh filename="package://edmo_snake_description/meshes/straight_connector_2_1.stl" scale="0.001 0.001 0.001"/>
@@ -166,5 +160,5 @@
   </visual>
   <collision>
-    <origin xyz="-${second_arm_x_offset} -0.0 -${arm_z_offset}" rpy="0 0 0"/>
+    <origin xyz="-0.222215 -0.014468 -0.02015" rpy="0 0 0"/>
     <geometry>
       <mesh filename="package://edmo_snake_description/meshes/straight_connector_2_1.stl" scale="0.001 0.001 0.001"/>
@@ -179,5 +173,5 @@
   </inertial>
   <visual>
-    <origin xyz="-${second_arm_x_offset} -0.0 -${arm_z_offset}" rpy="0 0 0"/>
+    <origin xyz="-0.227215 -0.014468 -0.02015" rpy="0 0 0"/>
     <geometry>
       <mesh filename="package://edmo_snake_description/meshes/base_3_1.stl" scale="0.001 0.001 0.001"/>
@@ -186,5 +180,5 @@
   </visual>
   <collision>
-    <origin xyz="-${second_arm_x_offset} -0.0 -${arm_z_offset}" rpy="0 0 0"/>
+    <origin xyz="-0.227215 -0.014468 -0.02015" rpy="0 0 0"/>
     <geometry>
       <mesh filename="package://edmo_snake_description/meshes/base_3_1.stl" scale="0.001 0.001 0.001"/>
@@ -199,5 +193,5 @@
   </inertial>
   <visual>
-    <origin xyz="-${second_arm_x_offset} -0.0 -${arm_z_offset}" rpy="0 0 0"/>
+    <origin xyz="-0.309015 0.003782 -0.02015" rpy="0 0 0"/>
     <geometry>
       <mesh filename="package://edmo_snake_description/meshes/cover_3_1.stl" scale="0.001 0.001 0.001"/>
@@ -206,5 +200,5 @@
   </visual>
   <collision>
-    <origin xyz="-${second_arm_x_offset} -0.0 -${arm_z_offset}" rpy="0 0 0"/>
+    <origin xyz="-0.309015 0.003782 -0.02015" rpy="0 0 0"/>
     <geometry>
       <mesh filename="package://edmo_snake_description/meshes/cover_3_1.stl" scale="0.001 0.001 0.001"/>
@@ -219,24 +213,23 @@
   </inertial>
   <visual>
-    <origin xyz="-${arm_x_offset} -0.0 -${arm_z_offset}" rpy="0 0 0"/>
-    <geometry>
-      <mesh filename="package://edmo_snake_description/meshes/arm_1_1.stl" scale="0.001 0.001 0.001"/>
-    </geometry>
-    <material name="silver"/>
-  </visual>
-  <collision>
-    <origin xyz="-${arm_x_offset} -0.0 -${arm_z_offset}" rpy="0 0 0"/>
-    <geometry>
-      <mesh filename="package://edmo_snake_description/meshes/arm_1_1.stl" scale="0.001 0.001 0.001"/>
+    <origin xyz="-0.304214 -0.307532 0.002883" rpy="0 0 0"/>
+    <geometry>
+      <mesh filename="package://edmo_snake_description/meshes/arm_3_1.stl" scale="0.001 0.001 0.001"/>
+    </geometry>
+    <material name="silver"/>
+  </visual>
+  <collision>
+    <origin xyz="-0.304214 -0.307532 0.002883" rpy="0 0 0"/>
+    <geometry>
+      <mesh filename="package://edmo_snake_description/meshes/arm_3_1.stl" scale="0.001 0.001 0.001"/>
     </geometry>
   </collision>
 </link>
 <joint name="dummy_joint" type="fixed">
-  <origin xyz="0.0 0.0 0.0" rpy="0 0 0"/>
   <parent link="dummy"/>
   <child link="base_link"/>
 </joint>
 <joint name="Rev1" type="continuous">
-  <origin xyz="${arm_x_offset} 0.0 ${arm_z_offset}" rpy="0 0 0"/>
+  <origin xyz="0.038414 0.041832 -0.002983" rpy="0 0 0"/>
   <parent link="base_link"/>
   <child link="arm_1_1"/>
@@ -244,25 +237,25 @@
 </joint>
 <joint name="Rigid2" type="fixed">
-  <origin xyz="0.0 -0.0 ${cover_z_offset}" rpy="0 0 0"/>
+  <origin xyz="0.043315 -0.003782 0.02005" rpy="0 0 0"/>
   <parent link="base_link"/>
   <child link="cover_1_1"/>
 </joint>
 <joint name="Rigid3" type="fixed">
-  <origin xyz="-${arm_x_offset} -0.0 -${arm_z_offset}" rpy="0 0 0"/>
+  <origin xyz="0.050951 -0.027364 0.023083" rpy="0 0 0"/>
   <parent link="arm_1_1"/>
   <child link="straight_connector_1_1"/>
 </joint>
 <joint name="Rigid5" type="fixed">
-  <origin xyz="-${arm_x_offset} -0.0 -${arm_z_offset}" rpy="0 0 0"/>
+  <origin xyz="0.055951 -0.027364 0.023083" rpy="0 0 0"/>
   <parent link="arm_1_1"/>
   <child link="base_2_1"/>
 </joint>
 <joint name="Rigid7" type="fixed">
-  <origin xyz="0.0 -0.0 0.0" rpy="0 0 0"/>
+  <origin xyz="0.0818 -0.01825 0.0" rpy="0 0 0"/>
   <parent link="base_2_1"/>
   <child link="cover_2_1"/>
 </joint>
 <joint name="Rev8" type="continuous">
-  <origin xyz="${second_arm_x_offset} 0.0 ${arm_z_offset}" rpy="0 0 0"/>
+  <origin xyz="0.076949 0.160214 -0.023033" rpy="0 0 0"/>
   <parent link="base_2_1"/>
   <child link="arm_2_1"/>
@@ -270,20 +263,20 @@
 </joint>
 <joint name="Rigid9" type="fixed">
-  <origin xyz="0.0 -0.0 0.0" rpy="0 0 0"/>
+  <origin xyz="0.050901 -0.160214 0.023083" rpy="0 0 0"/>
   <parent link="arm_2_1"/>
   <child link="straight_connector_2_1"/>
 </joint>
 <joint name="Rigid10" type="fixed">
-  <origin xyz="0.0 -0.0 0.0" rpy="0 0 0"/>
+  <origin xyz="0.055901 -0.160214 0.023083" rpy="0 0 0"/>
   <parent link="arm_2_1"/>
   <child link="base_3_1"/>
 </joint>
 <joint name="Rigid12" type="fixed">
-  <origin xyz="0.0 -0.0 0.0" rpy="0 0 0"/>
+  <origin xyz="0.0818 -0.01825 0.0" rpy="0 0 0"/>
   <parent link="base_3_1"/>
   <child link="cover_3_1"/>
 </joint>
 <joint name="Rev13" type="continuous">
-  <origin xyz="${second_arm_x_offset-arm_x_offset} 0.0 0.0" rpy="0 0 0"/>
+  <origin xyz="0.076999 0.293064 -0.023033" rpy="0 0 0"/>
   <parent link="base_3_1"/>
   <child link="arm_3_1"/>
