Commit message: create simulation launch and fix inertia for base

File: src/edmo_snake_description/urdf/edmo_snake_updated_backup.xacro (robot description, xacro)
@@ -4,7 +4,5 @@
 <xacro:include filename="$(find edmo_snake_description)/urdf/edmo_snake.trans" />
 <xacro:include filename="$(find edmo_snake_description)/urdf/edmo_snake.gazebo" />
-<xacro:property name="base_x_offset" value="0.005" />
-<xacro:property name="base_y_offset" value="0.015" />
-<xacro:property name="base_z_offset" value="0.02" />
+<xacro:property name="base_y_offset" value="0.02" />
 <xacro:property name="arm_x_offset" value="0.027" />
 <xacro:property name="arm_z_offset" value="0.02" />
@@ -16,11 +14,10 @@
 <link name="base_link">
   <inertial>
-    <origin xyz="-0.0 0.0 0.0" rpy="0 0 0"/>
+    <origin xyz="-0.005007218473459374 0.012097251893188315 0.016720619639640767" rpy="0 0 0"/>
     <mass value="0.03847845253485034"/>
-    <inertia  ixx="0.000019973523403298565" ixy="0" ixz="0" iyy="0.00002704471032440412" iyz="0" izz="0.000041246465847475135" />
-    <!-- <inertia ixx="2.2e-05" iyy="3.3e-05" izz="4.9e-05" ixy="2e-06" iyz="0.0" ixz="3e-06"/> -->
-  </inertial>
-  <visual>
-    <origin xyz="-${base_x_offset} -${base_y_offset} -${base_z_offset}" rpy="0 0 0"/>
+    <inertia ixx="2.2e-05" iyy="3.3e-05" izz="4.9e-05" ixy="2e-06" iyz="0.0" ixz="3e-06"/>
+  </inertial>
+  <visual>
+    <origin xyz="0 0 0" rpy="0 0 0"/>
     <geometry>
       <mesh filename="package://edmo_snake_description/meshes/base_link.stl" scale="0.001 0.001 0.001"/>
@@ -29,5 +26,5 @@
   </visual>
   <collision>
-    <origin xyz="${base_x_offset} -${base_y_offset} -${base_z_offset}" rpy="0 0 0"/>
+    <origin xyz="0 0 0" rpy="0 0 0"/>
     <geometry>
       <mesh filename="package://edmo_snake_description/meshes/base_link.stl" scale="0.001 0.001 0.001"/>
@@ -35,9 +32,9 @@
   </collision>
 </link>
-<!-- <link name="arm_1_1">
-  <inertial>
-    <origin xyz="-${arm_x_offset} -0.0 -${arm_z_offset}" rpy="0 0 0"/>
+<link name="arm_1_1">
+  <inertial>
+    <origin xyz="0.01945776199314793 -0.027540516201431886 0.02290733232110153" rpy="0 0 0"/>
     <mass value="0.03728860045356832"/>
-    <inertia  ixx="0.02105608333333333" ixy="0" ixz="0" iyy="0.03001933333333333" iyz="0" izz="0.04552541666666666" />
+    <inertia ixx="4.1e-05" iyy="3.7e-05" izz="7.3e-05" ixy="0.0" iyz="0.0" ixz="0.0"/>
   </inertial>
   <visual>
@@ -57,83 +54,83 @@
 <link name="cover_1_1">
   <inertial>
+    <origin xyz="-0.024705167127436287 0.01692961887353248 0.008504948193972128" rpy="0 0 0"/>
+    <mass value="0.014555566232575165"/>
+    <inertia ixx="3e-06" iyy="8e-06" izz="1e-05" ixy="-0.0" iyz="0.0" ixz="-0.0"/>
+  </inertial>
+  <visual>
     <origin xyz="-0.0 0.0 -${cover_z_offset}" rpy="0 0 0"/>
+    <geometry>
+      <mesh filename="package://edmo_snake_description/meshes/cover_1_1.stl" scale="0.001 0.001 0.001"/>
+    </geometry>
+    <material name="silver"/>
+  </visual>
+  <collision>
+    <origin xyz="-0.0 0.0 -${cover_z_offset}" rpy="0 0 0"/>
+    <geometry>
+      <mesh filename="package://edmo_snake_description/meshes/cover_1_1.stl" scale="0.001 0.001 0.001"/>
+    </geometry>
+  </collision>
+</link>
+<link name="straight_connector_1_1">
+  <inertial>
+    <origin xyz="0.002551839107067355 -3.695547974580382e-07 0.007885618930935433" rpy="0 0 0"/>
+    <mass value="0.007137238748366013"/>
+    <inertia ixx="2e-06" iyy="1e-06" izz="1e-06" ixy="-0.0" iyz="0.0" ixz="-0.0"/>
+  </inertial>
+  <visual>
+    <origin xyz="0.0 0.0 0.0" rpy="0 0 0"/>
+    <geometry>
+      <mesh filename="package://edmo_snake_description/meshes/straight_connector_1_1.stl" scale="0.001 0.001 0.001"/>
+    </geometry>
+    <material name="silver"/>
+  </visual>
+  <collision>
+    <origin xyz="0.0 0.0 0.0" rpy="0 0 0"/>
+    <geometry>
+      <mesh filename="package://edmo_snake_description/meshes/straight_connector_1_1.stl" scale="0.001 0.001 0.001"/>
+    </geometry>
+  </collision>
+</link>
+<link name="base_2_1">
+  <inertial>
+    <origin xyz="0.03347778152654057 -0.0023707481068117025 -0.0033293803603586837" rpy="0 0 0"/>
+    <mass value="0.03847845253485034"/>
+    <inertia ixx="2.2e-05" iyy="3.3e-05" izz="4.9e-05" ixy="2e-06" iyz="0.0" ixz="3e-06"/>
+  </inertial>
+  <visual>
+    <origin xyz="-0.0 -0.0 -0.0" rpy="0 0 0"/>
+    <geometry>
+      <mesh filename="package://edmo_snake_description/meshes/base_2_1.stl" scale="0.001 0.001 0.001"/>
+    </geometry>
+    <material name="silver"/>
+  </visual>
+  <collision>
+    <origin xyz="-0.0 -0.0 -0.0" rpy="0 0 0"/>
+    <geometry>
+      <mesh filename="package://edmo_snake_description/meshes/base_2_1.stl" scale="0.001 0.001 0.001"/>
+    </geometry>
+  </collision>
+</link>
+<link name="cover_2_1">
+  <inertial>
+    <origin xyz="-0.0247051671274362 0.016929618873532466 0.008504948193972663" rpy="0 0 0"/>
     <mass value="0.014555566232575165"/>
-    <inertia  ixx="0.002728125" ixy="0" ixz="0" iyy="0.0046378125" iyz="0" izz="0.0068203125" />
-  </inertial>
-  <visual>
-    <origin xyz="-0.0 0.0 -${cover_z_offset}" rpy="0 0 0"/>
-    <geometry>
-      <mesh filename="package://edmo_snake_description/meshes/cover_1_1.stl" scale="0.001 0.001 0.001"/>
-    </geometry>
-    <material name="silver"/>
-  </visual>
-  <collision>
-    <origin xyz="-0.0 0.0 -${cover_z_offset}" rpy="0 0 0"/>
-    <geometry>
-      <mesh filename="package://edmo_snake_description/meshes/cover_1_1.stl" scale="0.001 0.001 0.001"/>
-    </geometry>
-  </collision>
-</link>
-<link name="straight_connector_1_1">
-  <inertial>
-    <origin xyz="0.0 0.0 0.0" rpy="0 0 0"/>
-    <mass value="0.007137238748366013"/>
-    <inertia  ixx="0.0019556595095858954" ixy="0" ixz="0" iyy="0.0008469443550060953" iyz="0" izz="0.001416742979526397" />
-  </inertial>
-  <visual>
-    <origin xyz="0.0 0.0 0.0" rpy="0 0 0"/>
-    <geometry>
-      <mesh filename="package://edmo_snake_description/meshes/straight_connector_1_1.stl" scale="0.001 0.001 0.001"/>
-    </geometry>
-    <material name="silver"/>
-  </visual>
-  <collision>
-    <origin xyz="0.0 0.0 0.0" rpy="0 0 0"/>
-    <geometry>
-      <mesh filename="package://edmo_snake_description/meshes/straight_connector_1_1.stl" scale="0.001 0.001 0.001"/>
-    </geometry>
-  </collision>
-</link>
-<link name="base_2_1">
-  <inertial>
-    <origin xyz="-0.0 -0.0 -0.0" rpy="0 0 0"/>
-    <mass value="0.03847845253485034"/>
-    <inertia  ixx="0.01972516666666667" ixy="0" ixz="0" iyy="0.026708424150187243" iyz="0" izz="0.040733590816853904" />
-  </inertial>
-  <visual>
-    <origin xyz="-0.0 -0.0 -0.0" rpy="0 0 0"/>
-    <geometry>
-      <mesh filename="package://edmo_snake_description/meshes/base_2_1.stl" scale="0.001 0.001 0.001"/>
-    </geometry>
-    <material name="silver"/>
-  </visual>
-  <collision>
-    <origin xyz="-0.0 -0.0 -0.0" rpy="0 0 0"/>
-    <geometry>
-      <mesh filename="package://edmo_snake_description/meshes/base_2_1.stl" scale="0.001 0.001 0.001"/>
-    </geometry>
-  </collision>
-</link>
-<link name="cover_2_1">
-  <inertial>
+    <inertia ixx="3e-06" iyy="8e-06" izz="1e-05" ixy="-0.0" iyz="0.0" ixz="-0.0"/>
+  </inertial>
+  <visual>
     <origin xyz="-0.0 0.0 -0.0" rpy="0 0 0"/>
-    <mass value="0.014555566232575165"/>
-    <inertia  ixx="0.002728125" ixy="0" ixz="0" iyy="0.0046378125" iyz="0" izz="0.0068203125" />
-  </inertial>
-  <visual>
+    <geometry>
+      <mesh filename="package://edmo_snake_description/meshes/cover_2_1.stl" scale="0.001 0.001 0.001"/>
+    </geometry>
+    <material name="silver"/>
+  </visual>
+  <collision>
     <origin xyz="-0.0 0.0 -0.0" rpy="0 0 0"/>
     <geometry>
       <mesh filename="package://edmo_snake_description/meshes/cover_2_1.stl" scale="0.001 0.001 0.001"/>
     </geometry>
-    <material name="silver"/>
-  </visual>
-  <collision>
-    <origin xyz="-0.0 0.0 -0.0" rpy="0 0 0"/>
-    <geometry>
-      <mesh filename="package://edmo_snake_description/meshes/cover_2_1.stl" scale="0.001 0.001 0.001"/>
-    </geometry>
-  </collision>
-</link> -->
-<!-- <link name="arm_2_1">
+  </collision>
+</link>
+<link name="arm_2_1">
   <inertial>
     <origin xyz="0.019407761993148254 -0.16039051620143224 0.02290733232110207" rpy="0 0 0"/>
@@ -234,5 +231,5 @@
     </geometry>
   </collision>
-</link> -->
+</link>
 <joint name="dummy_joint" type="fixed">
   <origin xyz="0.0 0.0 0.0" rpy="0 0 0"/>
@@ -240,5 +237,5 @@
   <child link="base_link"/>
 </joint>
-<!-- <joint name="Rev1" type="continuous">
+<joint name="Rev1" type="continuous">
   <origin xyz="${arm_x_offset} 0.0 ${arm_z_offset}" rpy="0 0 0"/>
   <parent link="base_link"/>
@@ -265,6 +262,6 @@
   <parent link="base_2_1"/>
   <child link="cover_2_1"/>
-</joint> -->
-<!-- <joint name="Rev8" type="continuous">
+</joint>
+<joint name="Rev8" type="continuous">
   <origin xyz="${second_arm_x_offset} 0.0 ${arm_z_offset}" rpy="0 0 0"/>
   <parent link="base_2_1"/>
@@ -293,4 +290,3 @@
   <axis xyz="-0.0 1.0 -0.0"/>
 </joint>
- -->
 </robot>
