Commit message: set up correct TF tree and compute correct inertia tensors

File: src/edmo_snake_description/urdf/edmo_snake.xacro (robot description, xacro)
@@ -4,20 +4,21 @@
 <xacro:include filename="$(find edmo_snake_description)/urdf/edmo_snake.trans" />
 <xacro:include filename="$(find edmo_snake_description)/urdf/edmo_snake.gazebo" />
-<xacro:property name="base_x_offset" value="0.005" />
+<xacro:property name="base_x_offset" value="0.0" />
 <xacro:property name="base_y_offset" value="0.015" />
 <xacro:property name="base_z_offset" value="0.02" />
 <xacro:property name="arm_x_offset" value="0.027" />
 <xacro:property name="arm_z_offset" value="0.02" />
+<xacro:property name="cover_x_offset" value="0.02" />
 <xacro:property name="cover_z_offset" value="0.02" />
 <xacro:property name="straight_connector_x_offset" value="0.06" />
-<xacro:property name="second_arm_x_offset" value="0.16" />
+<xacro:property name="second_arm_x_offset" value="0.106" />
+<xacro:property name="arm_x_intertia_offset" value="0.03" />
 <link name="dummy">
 </link>
 <link name="base_link">
   <inertial>
-    <origin xyz="-0.0 0.0 0.0" rpy="0 0 0"/>
+    <origin xyz="0.0 0.0 0.0" rpy="0 0 0"/>
     <mass value="0.03847845253485034"/>
-    <inertia  ixx="0.000019973523403298565" ixy="0" ixz="0" iyy="0.00002704471032440412" iyz="0" izz="0.000041246465847475135" />
-    <!-- <inertia ixx="2.2e-05" iyy="3.3e-05" izz="4.9e-05" ixy="2e-06" iyz="0.0" ixz="3e-06"/> -->
+    <inertia ixx="0.000019973523403298565" ixy="0" ixz="0" iyy="0.00002704471032440412" iyz="0" izz="0.000041246465847475135" />
   </inertial>
   <visual>
@@ -35,19 +36,19 @@
   </collision>
 </link>
-<!-- <link name="arm_1_1">
-  <inertial>
-    <origin xyz="-${arm_x_offset} -0.0 -${arm_z_offset}" rpy="0 0 0"/>
+<link name="arm_1_1">
+  <inertial>
+    <origin xyz="${arm_x_intertia_offset} 0.0 0.0" rpy="0 0 0"/>
     <mass value="0.03728860045356832"/>
-    <inertia  ixx="0.02105608333333333" ixy="0" ixz="0" iyy="0.03001933333333333" iyz="0" izz="0.04552541666666666" />
-  </inertial>
-  <visual>
-    <origin xyz="-${arm_x_offset} -0.0 -${arm_z_offset}" rpy="0 0 0"/>
-    <geometry>
-      <mesh filename="package://edmo_snake_description/meshes/arm_1_1.stl" scale="0.001 0.001 0.001"/>
-    </geometry>
-    <material name="silver"/>
-  </visual>
-  <collision>
-    <origin xyz="-${arm_x_offset} -0.0 -${arm_z_offset}" rpy="0 0 0"/>
+    <inertia ixx="0.00002105608333333333" ixy="0" ixz="0" iyy="0.00003001933333333333" iyz="0" izz="0.00004552541666666666" />
+  </inertial>
+  <visual>
+    <origin xyz="-${arm_x_offset} -${base_y_offset} -${arm_z_offset}" rpy="0 0 0"/>
+    <geometry>
+      <mesh filename="package://edmo_snake_description/meshes/arm_1_1.stl" scale="0.001 0.001 0.001"/>
+    </geometry>
+    <material name="silver"/>
+  </visual>
+  <collision>
+    <origin xyz="-${arm_x_offset} -${base_y_offset} -${arm_z_offset}" rpy="0 0 0"/>
     <geometry>
       <mesh filename="package://edmo_snake_description/meshes/arm_1_1.stl" scale="0.001 0.001 0.001"/>
@@ -57,17 +58,17 @@
 <link name="cover_1_1">
   <inertial>
-    <origin xyz="-0.0 0.0 -${cover_z_offset}" rpy="0 0 0"/>
+    <origin xyz="0.0 0.0 0.0" rpy="0 0 0"/>
     <mass value="0.014555566232575165"/>
-    <inertia  ixx="0.002728125" ixy="0" ixz="0" iyy="0.0046378125" iyz="0" izz="0.0068203125" />
-  </inertial>
-  <visual>
-    <origin xyz="-0.0 0.0 -${cover_z_offset}" rpy="0 0 0"/>
-    <geometry>
-      <mesh filename="package://edmo_snake_description/meshes/cover_1_1.stl" scale="0.001 0.001 0.001"/>
-    </geometry>
-    <material name="silver"/>
-  </visual>
-  <collision>
-    <origin xyz="-0.0 0.0 -${cover_z_offset}" rpy="0 0 0"/>
+    <inertia ixx="0.000002728125" ixy="0" ixz="0" iyy="0.0000046378125" iyz="0" izz="0.0000068203125" />
+  </inertial>
+  <visual>
+    <origin xyz="-${cover_x_offset} -${base_y_offset} -${cover_z_offset}" rpy="0 0 0"/>
+    <geometry>
+      <mesh filename="package://edmo_snake_description/meshes/cover_1_1.stl" scale="0.001 0.001 0.001"/>
+    </geometry>
+    <material name="silver"/>
+  </visual>
+  <collision>
+    <origin xyz="-${cover_x_offset} -${base_y_offset} -${cover_z_offset}" rpy="0 0 0"/>
     <geometry>
       <mesh filename="package://edmo_snake_description/meshes/cover_1_1.stl" scale="0.001 0.001 0.001"/>
@@ -79,15 +80,15 @@
     <origin xyz="0.0 0.0 0.0" rpy="0 0 0"/>
     <mass value="0.007137238748366013"/>
-    <inertia  ixx="0.0019556595095858954" ixy="0" ixz="0" iyy="0.0008469443550060953" iyz="0" izz="0.001416742979526397" />
-  </inertial>
-  <visual>
-    <origin xyz="0.0 0.0 0.0" rpy="0 0 0"/>
-    <geometry>
-      <mesh filename="package://edmo_snake_description/meshes/straight_connector_1_1.stl" scale="0.001 0.001 0.001"/>
-    </geometry>
-    <material name="silver"/>
-  </visual>
-  <collision>
-    <origin xyz="0.0 0.0 0.0" rpy="0 0 0"/>
+    <inertia ixx="0.0000019556595095858954" ixy="0" ixz="0" iyy="0.0000008469443550060953" iyz="0" izz="0.000001416742979526397" />
+  </inertial>
+  <visual>
+    <origin xyz="-${straight_connector_x_offset+arm_x_offset} -${base_y_offset} -${base_z_offset}" rpy="0 0 0"/>
+    <geometry>
+      <mesh filename="package://edmo_snake_description/meshes/straight_connector_1_1.stl" scale="0.001 0.001 0.001"/>
+    </geometry>
+    <material name="silver"/>
+  </visual>
+  <collision>
+    <origin xyz="-${straight_connector_x_offset+arm_x_offset} -${base_y_offset} -${base_z_offset}" rpy="0 0 0"/>
     <geometry>
       <mesh filename="package://edmo_snake_description/meshes/straight_connector_1_1.stl" scale="0.001 0.001 0.001"/>
@@ -97,19 +98,19 @@
 <link name="base_2_1">
   <inertial>
-    <origin xyz="-0.0 -0.0 -0.0" rpy="0 0 0"/>
+    <origin xyz="0.0 0.0 0.0" rpy="0 0 0"/>
     <mass value="0.03847845253485034"/>
-    <inertia  ixx="0.01972516666666667" ixy="0" ixz="0" iyy="0.026708424150187243" iyz="0" izz="0.040733590816853904" />
-  </inertial>
-  <visual>
-    <origin xyz="-0.0 -0.0 -0.0" rpy="0 0 0"/>
-    <geometry>
-      <mesh filename="package://edmo_snake_description/meshes/base_2_1.stl" scale="0.001 0.001 0.001"/>
-    </geometry>
-    <material name="silver"/>
-  </visual>
-  <collision>
-    <origin xyz="-0.0 -0.0 -0.0" rpy="0 0 0"/>
-    <geometry>
-      <mesh filename="package://edmo_snake_description/meshes/base_2_1.stl" scale="0.001 0.001 0.001"/>
+    <inertia ixx="0.000019973523403298565" ixy="0" ixz="0" iyy="0.00002704471032440412" iyz="0" izz="0.000041246465847475135" />
+  </inertial>
+  <visual>
+    <origin xyz="0.0 -${base_y_offset} -${base_z_offset}" rpy="0 0 0"/>
+    <geometry>
+      <mesh filename="package://edmo_snake_description/meshes/base_link.stl" scale="0.001 0.001 0.001"/>
+    </geometry>
+    <material name="silver"/>
+  </visual>
+  <collision>
+    <origin xyz="0.0 -${base_y_offset} -${base_z_offset}" rpy="0 0 0"/>
+    <geometry>
+      <mesh filename="package://edmo_snake_description/meshes/base_link.stl" scale="0.001 0.001 0.001"/>
     </geometry>
   </collision>
@@ -117,37 +118,37 @@
 <link name="cover_2_1">
   <inertial>
-    <origin xyz="-0.0 0.0 -0.0" rpy="0 0 0"/>
+    <origin xyz="0.0 0.0 0.0" rpy="0 0 0"/>
     <mass value="0.014555566232575165"/>
-    <inertia  ixx="0.002728125" ixy="0" ixz="0" iyy="0.0046378125" iyz="0" izz="0.0068203125" />
-  </inertial>
-  <visual>
-    <origin xyz="-0.0 0.0 -0.0" rpy="0 0 0"/>
-    <geometry>
-      <mesh filename="package://edmo_snake_description/meshes/cover_2_1.stl" scale="0.001 0.001 0.001"/>
-    </geometry>
-    <material name="silver"/>
-  </visual>
-  <collision>
-    <origin xyz="-0.0 0.0 -0.0" rpy="0 0 0"/>
-    <geometry>
-      <mesh filename="package://edmo_snake_description/meshes/cover_2_1.stl" scale="0.001 0.001 0.001"/>
-    </geometry>
-  </collision>
-</link> -->
-<!-- <link name="arm_2_1">
-  <inertial>
-    <origin xyz="0.019407761993148254 -0.16039051620143224 0.02290733232110207" rpy="0 0 0"/>
+    <inertia ixx="0.000002728125" ixy="0" ixz="0" iyy="0.0000046378125" iyz="0" izz="0.0000068203125" />
+  </inertial>
+  <visual>
+    <origin xyz="-${cover_x_offset} -${base_y_offset} -${cover_z_offset}" rpy="0 0 0"/>
+    <geometry>
+      <mesh filename="package://edmo_snake_description/meshes/cover_1_1.stl" scale="0.001 0.001 0.001"/>
+    </geometry>
+    <material name="silver"/>
+  </visual>
+  <collision>
+    <origin xyz="-${cover_x_offset} -${base_y_offset} -${cover_z_offset}" rpy="0 0 0"/>
+    <geometry>
+      <mesh filename="package://edmo_snake_description/meshes/cover_1_1.stl" scale="0.001 0.001 0.001"/>
+    </geometry>
+  </collision>
+</link>
+<link name="arm_2_1">
+  <inertial>
+    <origin xyz="${arm_x_intertia_offset} 0.0 0.0" rpy="0 0 0"/>
     <mass value="0.03728860045356832"/>
-    <inertia ixx="4.1e-05" iyy="3.7e-05" izz="7.3e-05" ixy="0.0" iyz="0.0" ixz="0.0"/>
-  </inertial>
-  <visual>
-    <origin xyz="-${arm_x_offset} -0.0 -${arm_z_offset}" rpy="0 0 0"/>
-    <geometry>
-      <mesh filename="package://edmo_snake_description/meshes/arm_1_1.stl" scale="0.001 0.001 0.001"/>
-    </geometry>
-    <material name="silver"/>
-  </visual>
-  <collision>
-    <origin xyz="-${arm_x_offset} -0.0 -${arm_z_offset}" rpy="0 0 0"/>
+    <inertia ixx="0.00002105608333333333" ixy="0" ixz="0" iyy="0.00003001933333333333" iyz="0" izz="0.00004552541666666666" />
+  </inertial>
+  <visual>
+    <origin xyz="-${arm_x_offset} -${base_y_offset} -${arm_z_offset}" rpy="0 0 0"/>
+    <geometry>
+      <mesh filename="package://edmo_snake_description/meshes/arm_1_1.stl" scale="0.001 0.001 0.001"/>
+    </geometry>
+    <material name="silver"/>
+  </visual>
+  <collision>
+    <origin xyz="-${arm_x_offset} -${base_y_offset} -${arm_z_offset}" rpy="0 0 0"/>
     <geometry>
       <mesh filename="package://edmo_snake_description/meshes/arm_1_1.stl" scale="0.001 0.001 0.001"/>
@@ -157,19 +158,19 @@
 <link name="straight_connector_2_1">
   <inertial>
-    <origin xyz="0.002551839107067605 -3.6955479817100956e-07 0.007885618930935943" rpy="0 0 0"/>
+    <origin xyz="0.0 0.0 0.0" rpy="0 0 0"/>
     <mass value="0.007137238748366013"/>
-    <inertia ixx="2e-06" iyy="1e-06" izz="1e-06" ixy="-0.0" iyz="0.0" ixz="-0.0"/>
-  </inertial>
-  <visual>
-    <origin xyz="-${second_arm_x_offset} -0.0 -${arm_z_offset}" rpy="0 0 0"/>
-    <geometry>
-      <mesh filename="package://edmo_snake_description/meshes/straight_connector_2_1.stl" scale="0.001 0.001 0.001"/>
-    </geometry>
-    <material name="silver"/>
-  </visual>
-  <collision>
-    <origin xyz="-${second_arm_x_offset} -0.0 -${arm_z_offset}" rpy="0 0 0"/>
-    <geometry>
-      <mesh filename="package://edmo_snake_description/meshes/straight_connector_2_1.stl" scale="0.001 0.001 0.001"/>
+    <inertia ixx="0.0000019556595095858954" ixy="0" ixz="0" iyy="0.0000008469443550060953" iyz="0" izz="0.000001416742979526397" />
+  </inertial>
+  <visual>
+    <origin xyz="-${straight_connector_x_offset+arm_x_offset} -${base_y_offset} -${base_z_offset}" rpy="0 0 0"/>
+    <geometry>
+      <mesh filename="package://edmo_snake_description/meshes/straight_connector_1_1.stl" scale="0.001 0.001 0.001"/>
+    </geometry>
+    <material name="silver"/>
+  </visual>
+  <collision>
+    <origin xyz="-${straight_connector_x_offset+arm_x_offset} -${base_y_offset} -${base_z_offset}" rpy="0 0 0"/>
+    <geometry>
+      <mesh filename="package://edmo_snake_description/meshes/straight_connector_1_1.stl" scale="0.001 0.001 0.001"/>
     </geometry>
   </collision>
@@ -177,19 +178,19 @@
 <link name="base_3_1">
   <inertial>
-    <origin xyz="0.03347778152654096 -0.00237074810681245 -0.003329380360358153" rpy="0 0 0"/>
+    <origin xyz="0.0 0.0 0.0" rpy="0 0 0"/>
     <mass value="0.03847845253485034"/>
-    <inertia ixx="2.2e-05" iyy="3.3e-05" izz="4.9e-05" ixy="2e-06" iyz="0.0" ixz="3e-06"/>
-  </inertial>
-  <visual>
-    <origin xyz="-${second_arm_x_offset} -0.0 -${arm_z_offset}" rpy="0 0 0"/>
-    <geometry>
-      <mesh filename="package://edmo_snake_description/meshes/base_3_1.stl" scale="0.001 0.001 0.001"/>
-    </geometry>
-    <material name="silver"/>
-  </visual>
-  <collision>
-    <origin xyz="-${second_arm_x_offset} -0.0 -${arm_z_offset}" rpy="0 0 0"/>
-    <geometry>
-      <mesh filename="package://edmo_snake_description/meshes/base_3_1.stl" scale="0.001 0.001 0.001"/>
+    <inertia ixx="0.000019973523403298565" ixy="0" ixz="0" iyy="0.00002704471032440412" iyz="0" izz="0.000041246465847475135" />
+  </inertial>
+  <visual>
+    <origin xyz="0.0 -${base_y_offset} -${base_z_offset}" rpy="0 0 0"/>
+    <geometry>
+      <mesh filename="package://edmo_snake_description/meshes/base_link.stl" scale="0.001 0.001 0.001"/>
+    </geometry>
+    <material name="silver"/>
+  </visual>
+  <collision>
+    <origin xyz="0.0 -${base_y_offset} -${base_z_offset}" rpy="0 0 0"/>
+    <geometry>
+      <mesh filename="package://edmo_snake_description/meshes/base_link.stl" scale="0.001 0.001 0.001"/>
     </geometry>
   </collision>
@@ -197,19 +198,19 @@
 <link name="cover_3_1">
   <inertial>
-    <origin xyz="-0.024705167127435923 0.01692961887353178 0.0085049481939732" rpy="0 0 0"/>
+    <origin xyz="0.0 0.0 0.0" rpy="0 0 0"/>
     <mass value="0.014555566232575165"/>
-    <inertia ixx="3e-06" iyy="8e-06" izz="1e-05" ixy="-0.0" iyz="0.0" ixz="-0.0"/>
-  </inertial>
-  <visual>
-    <origin xyz="-${second_arm_x_offset} -0.0 -${arm_z_offset}" rpy="0 0 0"/>
-    <geometry>
-      <mesh filename="package://edmo_snake_description/meshes/cover_3_1.stl" scale="0.001 0.001 0.001"/>
-    </geometry>
-    <material name="silver"/>
-  </visual>
-  <collision>
-    <origin xyz="-${second_arm_x_offset} -0.0 -${arm_z_offset}" rpy="0 0 0"/>
-    <geometry>
-      <mesh filename="package://edmo_snake_description/meshes/cover_3_1.stl" scale="0.001 0.001 0.001"/>
+    <inertia ixx="0.000002728125" ixy="0" ixz="0" iyy="0.0000046378125" iyz="0" izz="0.0000068203125" />
+  </inertial>
+  <visual>
+    <origin xyz="-${cover_x_offset} -${base_y_offset} -${cover_z_offset}" rpy="0 0 0"/>
+    <geometry>
+      <mesh filename="package://edmo_snake_description/meshes/cover_1_1.stl" scale="0.001 0.001 0.001"/>
+    </geometry>
+    <material name="silver"/>
+  </visual>
+  <collision>
+    <origin xyz="-${cover_x_offset} -${base_y_offset} -${cover_z_offset}" rpy="0 0 0"/>
+    <geometry>
+      <mesh filename="package://edmo_snake_description/meshes/cover_1_1.stl" scale="0.001 0.001 0.001"/>
     </geometry>
   </collision>
@@ -217,22 +218,22 @@
 <link name="arm_3_1">
   <inertial>
-    <origin xyz="0.019357761993148204 -0.29324051620143254 0.022907332321102584" rpy="0 0 0"/>
+    <origin xyz="${arm_x_intertia_offset} 0.0 0.0" rpy="0 0 0"/>
     <mass value="0.03728860045356832"/>
-    <inertia ixx="4.1e-05" iyy="3.7e-05" izz="7.3e-05" ixy="0.0" iyz="0.0" ixz="0.0"/>
-  </inertial>
-  <visual>
-    <origin xyz="-${arm_x_offset} -0.0 -${arm_z_offset}" rpy="0 0 0"/>
-    <geometry>
-      <mesh filename="package://edmo_snake_description/meshes/arm_1_1.stl" scale="0.001 0.001 0.001"/>
-    </geometry>
-    <material name="silver"/>
-  </visual>
-  <collision>
-    <origin xyz="-${arm_x_offset} -0.0 -${arm_z_offset}" rpy="0 0 0"/>
-    <geometry>
-      <mesh filename="package://edmo_snake_description/meshes/arm_1_1.stl" scale="0.001 0.001 0.001"/>
-    </geometry>
-  </collision>
-</link> -->
+    <inertia ixx="0.00002105608333333333" ixy="0" ixz="0" iyy="0.00003001933333333333" iyz="0" izz="0.00004552541666666666" />
+  </inertial>
+  <visual>
+    <origin xyz="-${arm_x_offset} -${base_y_offset} -${arm_z_offset}" rpy="0 0 0"/>
+    <geometry>
+      <mesh filename="package://edmo_snake_description/meshes/arm_1_1.stl" scale="0.001 0.001 0.001"/>
+    </geometry>
+    <material name="silver"/>
+  </visual>
+  <collision>
+    <origin xyz="-${arm_x_offset} -${base_y_offset} -${arm_z_offset}" rpy="0 0 0"/>
+    <geometry>
+      <mesh filename="package://edmo_snake_description/meshes/arm_1_1.stl" scale="0.001 0.001 0.001"/>
+    </geometry>
+  </collision>
+</link>
 <joint name="dummy_joint" type="fixed">
   <origin xyz="0.0 0.0 0.0" rpy="0 0 0"/>
@@ -240,57 +241,56 @@
   <child link="base_link"/>
 </joint>
-<!-- <joint name="Rev1" type="continuous">
-  <origin xyz="${arm_x_offset} 0.0 ${arm_z_offset}" rpy="0 0 0"/>
+<joint name="Rev1" type="continuous">
+  <origin xyz="${arm_x_offset} 0.0 0.0" rpy="0 0 0"/>
   <parent link="base_link"/>
   <child link="arm_1_1"/>
-  <axis xyz="-0.0 1.0 -0.0"/>
+  <axis xyz="0.0 1.0 0.0"/>
 </joint>
 <joint name="Rigid2" type="fixed">
-  <origin xyz="0.0 -0.0 ${cover_z_offset}" rpy="0 0 0"/>
+  <origin xyz="${cover_x_offset} 0.0 0.0" rpy="0 0 0"/>
   <parent link="base_link"/>
   <child link="cover_1_1"/>
 </joint>
 <joint name="Rigid3" type="fixed">
-  <origin xyz="-${arm_x_offset} -0.0 -${arm_z_offset}" rpy="0 0 0"/>
+  <origin xyz="${straight_connector_x_offset} 0.0 0.0" rpy="0 0 0"/>
   <parent link="arm_1_1"/>
   <child link="straight_connector_1_1"/>
 </joint>
 <joint name="Rigid5" type="fixed">
-  <origin xyz="-${arm_x_offset} -0.0 -${arm_z_offset}" rpy="0 0 0"/>
+  <origin xyz="${second_arm_x_offset} 0.0 0.0" rpy="0 0 0"/>
   <parent link="arm_1_1"/>
   <child link="base_2_1"/>
 </joint>
 <joint name="Rigid7" type="fixed">
-  <origin xyz="0.0 -0.0 0.0" rpy="0 0 0"/>
+  <origin xyz="${cover_x_offset} 0.0 0.0" rpy="0 0 0"/>
   <parent link="base_2_1"/>
   <child link="cover_2_1"/>
-</joint> -->
-<!-- <joint name="Rev8" type="continuous">
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
Commit message: resolve intertia components for ABS plastic

File: src/edmo_snake_description/urdf/edmo_snake.xacro (robot description, xacro)
@@ -19,6 +19,6 @@
   <inertial>
     <origin xyz="0.0 0.0 0.0" rpy="0 0 0"/>
-    <mass value="0.03847845253485034"/>
-    <inertia ixx="0.000019973523403298565" ixy="0" ixz="0" iyy="0.00002704471032440412" iyz="0" izz="0.000041246465847475135" />
+    <mass value="0.040787"/>
+    <inertia ixx="0.000021171851916666665" ixy="0" ixz="0" iyy="0.000028667280707362297" iyz="0" izz="0.00004372108262402896" />
   </inertial>
   <visual>
@@ -39,6 +39,6 @@
   <inertial>
     <origin xyz="${arm_x_intertia_offset} 0.0 0.0" rpy="0 0 0"/>
-    <mass value="0.03728860045356832"/>
-    <inertia ixx="0.00002105608333333333" ixy="0" ixz="0" iyy="0.00003001933333333333" iyz="0" izz="0.00004552541666666666" />
+    <mass value="0.039526"/>
+    <inertia ixx="0.000022493587833333332" ixy="0" ixz="0" iyy="0.00003206876133333333" iyz="0" izz="0.00004863344916666667" />
   </inertial>
   <visual>
@@ -59,6 +59,6 @@
   <inertial>
     <origin xyz="0.0 0.0 0.0" rpy="0 0 0"/>
-    <mass value="0.014555566232575165"/>
-    <inertia ixx="0.000002728125" ixy="0" ixz="0" iyy="0.0000046378125" iyz="0" izz="0.0000068203125" />
+    <mass value="0.015429"/>
+    <inertia ixx="0.0000028929375" ixy="0" ixz="0" iyy="0.00000491799375" iyz="0" izz="0.00000723234375" />
   </inertial>
   <visual>
@@ -79,6 +79,6 @@
   <inertial>
     <origin xyz="0.0 0.0 0.0" rpy="0 0 0"/>
-    <mass value="0.007137238748366013"/>
-    <inertia ixx="0.0000019556595095858954" ixy="0" ixz="0" iyy="0.0000008469443550060953" iyz="0" izz="0.000001416742979526397" />
+    <mass value="0.007565"/>
+    <inertia ixx="0.000002074973939693871" ixy="0" ixz="0" iyy="0.0000008986162756831851" iyz="0" izz="0.0000015031782103951184" />
   </inertial>
   <visual>
@@ -99,6 +99,6 @@
   <inertial>
     <origin xyz="0.0 0.0 0.0" rpy="0 0 0"/>
-    <mass value="0.03847845253485034"/>
-    <inertia ixx="0.000019973523403298565" ixy="0" ixz="0" iyy="0.00002704471032440412" iyz="0" izz="0.000041246465847475135" />
+    <mass value="0.040787"/>
+    <inertia ixx="0.000021171851916666665" ixy="0" ixz="0" iyy="0.000028667280707362297" iyz="0" izz="0.00004372108262402896" />
   </inertial>
   <visual>
@@ -119,6 +119,6 @@
   <inertial>
     <origin xyz="0.0 0.0 0.0" rpy="0 0 0"/>
-    <mass value="0.014555566232575165"/>
-    <inertia ixx="0.000002728125" ixy="0" ixz="0" iyy="0.0000046378125" iyz="0" izz="0.0000068203125" />
+    <mass value="0.015429"/>
+    <inertia ixx="0.0000028929375" ixy="0" ixz="0" iyy="0.00000491799375" iyz="0" izz="0.00000723234375" />
   </inertial>
   <visual>
@@ -139,6 +139,6 @@
   <inertial>
     <origin xyz="${arm_x_intertia_offset} 0.0 0.0" rpy="0 0 0"/>
-    <mass value="0.03728860045356832"/>
-    <inertia ixx="0.00002105608333333333" ixy="0" ixz="0" iyy="0.00003001933333333333" iyz="0" izz="0.00004552541666666666" />
+    <mass value="0.039526"/>
+    <inertia ixx="0.000022493587833333332" ixy="0" ixz="0" iyy="0.00003206876133333333" iyz="0" izz="0.00004863344916666667" />
   </inertial>
   <visual>
@@ -159,6 +159,6 @@
   <inertial>
     <origin xyz="0.0 0.0 0.0" rpy="0 0 0"/>
-    <mass value="0.007137238748366013"/>
-    <inertia ixx="0.0000019556595095858954" ixy="0" ixz="0" iyy="0.0000008469443550060953" iyz="0" izz="0.000001416742979526397" />
+    <mass value="0.007565"/>
+    <inertia ixx="0.000002074973939693871" ixy="0" ixz="0" iyy="0.0000008986162756831851" iyz="0" izz="0.0000015031782103951184" />
   </inertial>
   <visual>
@@ -179,6 +179,6 @@
   <inertial>
     <origin xyz="0.0 0.0 0.0" rpy="0 0 0"/>
-    <mass value="0.03847845253485034"/>
-    <inertia ixx="0.000019973523403298565" ixy="0" ixz="0" iyy="0.00002704471032440412" iyz="0" izz="0.000041246465847475135" />
+    <mass value="0.040787"/>
+    <inertia ixx="0.000021171851916666665" ixy="0" ixz="0" iyy="0.000028667280707362297" iyz="0" izz="0.00004372108262402896" />
   </inertial>
   <visual>
@@ -199,6 +199,6 @@
   <inertial>
     <origin xyz="0.0 0.0 0.0" rpy="0 0 0"/>
-    <mass value="0.014555566232575165"/>
-    <inertia ixx="0.000002728125" ixy="0" ixz="0" iyy="0.0000046378125" iyz="0" izz="0.0000068203125" />
+    <mass value="0.015429"/>
+    <inertia ixx="0.0000028929375" ixy="0" ixz="0" iyy="0.00000491799375" iyz="0" izz="0.00000723234375" />
   </inertial>
   <visual>
@@ -219,6 +219,6 @@
   <inertial>
     <origin xyz="${arm_x_intertia_offset} 0.0 0.0" rpy="0 0 0"/>
-    <mass value="0.03728860045356832"/>
-    <inertia ixx="0.00002105608333333333" ixy="0" ixz="0" iyy="0.00003001933333333333" iyz="0" izz="0.00004552541666666666" />
+    <mass value="0.039526"/>
+    <inertia ixx="0.000022493587833333332" ixy="0" ixz="0" iyy="0.00003206876133333333" iyz="0" izz="0.00004863344916666667" />
   </inertial>
   <visual>
