Commit message: add clip connector to xacro model

File: src/edmo_snake_description/urdf/edmo_snake.xacro (robot description, xacro)
@@ -96,4 +96,24 @@
   </collision>
 </link>
+<link name="clip_connector_1_1">
+  <inertial>
+    <origin xyz="0.0 0.0 0.0" rpy="0 0 0"/>
+    <mass value="0.004143"/>
+    <inertia  ixx="0.0000008225581966461201" ixy="0" ixz="0" iyy="0.00000014973490050335027" iyz="0" izz="0.0000009247245608945109" />
+  </inertial>
+  <visual>
+    <origin xyz="-${straight_connector_x_offset+arm_x_offset} -${base_y_offset} -${base_z_offset}" rpy="0 0 0"/>
+    <geometry>
+      <mesh filename="package://edmo_snake_description/meshes/clip_connector_1_1.stl" scale="0.001 0.001 0.001"/>
+    </geometry>
+    <material name="silver"/>
+  </visual>
+  <collision>
+    <origin xyz="-${straight_connector_x_offset+arm_x_offset} -${base_y_offset} -${base_z_offset}" rpy="0 0 0"/>
+    <geometry>
+      <mesh filename="package://edmo_snake_description/meshes/clip_connector_1_1.stl" scale="0.001 0.001 0.001"/>
+    </geometry>
+  </collision>
+</link>
 <link name="base_2_1">
   <inertial>
@@ -176,4 +196,24 @@
   </collision>
 </link>
+<link name="clip_connector_2_1">
+  <inertial>
+    <origin xyz="0.0 0.0 0.0" rpy="0 0 0"/>
+    <mass value="0.004143"/>
+    <inertia  ixx="0.0000008225581966461201" ixy="0" ixz="0" iyy="0.00000014973490050335027" iyz="0" izz="0.0000009247245608945109" />
+  </inertial>
+  <visual>
+    <origin xyz="-${straight_connector_x_offset+arm_x_offset} -${base_y_offset} -${base_z_offset}" rpy="0 0 0"/>
+    <geometry>
+      <mesh filename="package://edmo_snake_description/meshes/clip_connector_1_1.stl" scale="0.001 0.001 0.001"/>
+    </geometry>
+    <material name="silver"/>
+  </visual>
+  <collision>
+    <origin xyz="-${straight_connector_x_offset+arm_x_offset} -${base_y_offset} -${base_z_offset}" rpy="0 0 0"/>
+    <geometry>
+      <mesh filename="package://edmo_snake_description/meshes/clip_connector_1_1.stl" scale="0.001 0.001 0.001"/>
+    </geometry>
+  </collision>
+</link>
 <link name="base_3_1">
   <inertial>
@@ -236,5 +276,5 @@
   </collision>
 </link>
-<joint name="dummy_joint" type="fixed">
+<joint name="Rigid0" type="fixed">
   <origin xyz="0.0 0.0 0.0" rpy="0 0 0"/>
   <parent link="dummy"/>
@@ -257,4 +297,9 @@
   <child link="straight_connector_1_1"/>
 </joint>
+<joint name="Rigid4" type="fixed">
+  <origin xyz="${straight_connector_x_offset} 0.0 0.0" rpy="0 0 0"/>
+  <parent link="arm_1_1"/>
+  <child link="clip_connector_1_1"/>
+</joint>
 <joint name="Rigid5" type="fixed">
   <origin xyz="${second_arm_x_offset} 0.0 0.0" rpy="0 0 0"/>
@@ -283,4 +328,9 @@
   <child link="base_3_1"/>
 </joint>
+<joint name="Rigid11" type="fixed">
+  <origin xyz="${straight_connector_x_offset} 0.0 0.0" rpy="0 0 0"/>
+  <parent link="arm_2_1"/>
+  <child link="clip_connector_2_1"/>
+</joint>
 <joint name="Rigid12" type="fixed">
   <origin xyz="${cover_x_offset} 0.0 0.0" rpy="0 0 0"/>

Commit message: add motors to edmo model

File: src/edmo_snake_description/urdf/edmo_snake.xacro (robot description, xacro)
@@ -13,4 +13,7 @@
 <xacro:property name="straight_connector_x_offset" value="0.06" />
 <xacro:property name="second_arm_x_offset" value="0.106" />
+<xacro:property name="motor_x_offset" value="0.018" />
+<xacro:property name="motor_y_offset" value="0.002" />
+<xacro:property name="motor_z_offset" value="0.0008" />
 <xacro:property name="arm_x_intertia_offset" value="0.03" />
 <link name="dummy">
@@ -273,4 +276,64 @@
     <geometry>
       <mesh filename="package://edmo_snake_description/meshes/arm_1_1.stl" scale="0.001 0.001 0.001"/>
+    </geometry>
+  </collision>
+</link>
+<link name="motor_box_1">
+  <inertial>
+    <origin xyz="0.0 0.0 0.0" rpy="0 0 0"/>
+    <mass value="0.057"/>
+    <inertia ixx="0.0000090309375" ixy="0" ixz="0" iyy="0.000008846874999999999" iyz="0" izz="0.000014265437499999999" />
+  </inertial>
+  <visual>
+    <origin xyz="0.003 -0.058 -0.01" rpy="0 0 0"/>
+    <geometry>
+      <mesh filename="package://edmo_snake_description/meshes/motor_box_1.stl" scale="0.001 0.001 0.001"/>
+    </geometry>
+    <material name="silver"/>
+  </visual>
+  <collision>
+    <origin xyz="0.003 -0.058 -0.01" rpy="0 0 0"/>
+    <geometry>
+      <mesh filename="package://edmo_snake_description/meshes/motor_box_1.stl" scale="0.001 0.001 0.001"/>
+    </geometry>
+  </collision>
+</link>
+<link name="motor_box_2">
+  <inertial>
+    <origin xyz="0.0 0.0 0.0" rpy="0 0 0"/>
+    <mass value="0.057"/>
+    <inertia ixx="0.0000090309375" ixy="0" ixz="0" iyy="0.000008846874999999999" iyz="0" izz="0.000014265437499999999" />
+  </inertial>
+  <visual>
+    <origin xyz="0.003 -0.058 -0.01" rpy="0 0 0"/>
+    <geometry>
+      <mesh filename="package://edmo_snake_description/meshes/motor_box_1.stl" scale="0.001 0.001 0.001"/>
+    </geometry>
+    <material name="silver"/>
+  </visual>
+  <collision>
+    <origin xyz="0.003 -0.058 -0.01" rpy="0 0 0"/>
+    <geometry>
+      <mesh filename="package://edmo_snake_description/meshes/motor_box_1.stl" scale="0.001 0.001 0.001"/>
+    </geometry>
+  </collision>
+</link>
+<link name="motor_box_3">
+  <inertial>
+    <origin xyz="0.0 0.0 0.0" rpy="0 0 0"/>
+    <mass value="0.057"/>
+    <inertia ixx="0.0000090309375" ixy="0" ixz="0" iyy="0.000008846874999999999" iyz="0" izz="0.000014265437499999999" />
+  </inertial>
+  <visual>
+    <origin xyz="0.003 -0.058 -0.01" rpy="0 0 0"/>
+    <geometry>
+      <mesh filename="package://edmo_snake_description/meshes/motor_box_1.stl" scale="0.001 0.001 0.001"/>
+    </geometry>
+    <material name="silver"/>
+  </visual>
+  <collision>
+    <origin xyz="0.003 -0.058 -0.01" rpy="0 0 0"/>
+    <geometry>
+      <mesh filename="package://edmo_snake_description/meshes/motor_box_1.stl" scale="0.001 0.001 0.001"/>
     </geometry>
   </collision>
@@ -344,3 +407,18 @@
   <axis xyz="0.0 1.0 0.0"/>
 </joint>
+<joint name="Rigid14" type="fixed">
+  <origin xyz="${motor_x_offset} ${motor_y_offset} ${motor_z_offset}" rpy="0 0 0"/>
+  <parent link="base_link"/>
+  <child link="motor_box_1"/>
+</joint>
+<joint name="Rigid15" type="fixed">
+  <origin xyz="${motor_x_offset} ${motor_y_offset} ${motor_z_offset}" rpy="0 0 0"/>
+  <parent link="base_2_1"/>
+  <child link="motor_box_2"/>
+</joint>
+<joint name="Rigid16" type="fixed">
+  <origin xyz="${motor_x_offset} ${motor_y_offset} ${motor_z_offset}" rpy="0 0 0"/>
+  <parent link="base_3_1"/>
+  <child link="motor_box_3"/>
+</joint>
 </robot>

Commit message: tune pid params and set joint safety limits

File: src/edmo_snake_description/urdf/edmo_snake.xacro (robot description, xacro)
@@ -344,9 +344,14 @@
   <child link="base_link"/>
 </joint>
-<joint name="Rev1" type="continuous">
+<joint name="Rev1" type="revolute">
   <origin xyz="${arm_x_offset} 0.0 0.0" rpy="0 0 0"/>
   <parent link="base_link"/>
   <child link="arm_1_1"/>
   <axis xyz="0.0 1.0 0.0"/>
+  <!-- Joint limits -->
+  <limit lower="-1.47"
+        upper="1.47"
+        effort="0.5"
+        velocity="0.5"/>
 </joint>
 <joint name="Rigid2" type="fixed">
@@ -375,9 +380,14 @@
   <child link="cover_2_1"/>
 </joint>
-<joint name="Rev8" type="continuous">
+<joint name="Rev8" type="revolute">
   <origin xyz="${arm_x_offset} 0.0 0.0" rpy="0 0 0"/>
   <parent link="base_2_1"/>
   <child link="arm_2_1"/>
   <axis xyz="0.0 1.0 0.0"/>
+  <!-- Joint limits -->
+  <limit lower="-1.47"
+        upper="1.47"
+        effort="0.5"
+        velocity="0.5"/>
 </joint>
 <joint name="Rigid9" type="fixed">
@@ -401,9 +411,14 @@
   <child link="cover_3_1"/>
 </joint>
-<joint name="Rev13" type="continuous">
+<joint name="Rev13" type="revolute">
   <origin xyz="${arm_x_offset} 0.0 0.0" rpy="0 0 0"/>
   <parent link="base_3_1"/>
   <child link="arm_3_1"/>
   <axis xyz="0.0 1.0 0.0"/>
+  <!-- Joint limits -->
+  <limit lower="-1.47"
+        upper="1.47"
+        effort="1.0"
+        velocity="0.2"/>
 </joint>
 <joint name="Rigid14" type="fixed">

Commit message: change friction and joint limits

File: src/edmo_snake_description/urdf/edmo_snake.xacro (robot description, xacro)
@@ -350,7 +350,7 @@
   <axis xyz="0.0 1.0 0.0"/>
   <!-- Joint limits -->
-  <limit lower="-1.47"
-        upper="1.47"
-        effort="0.5"
+  <limit lower="-2.00"
+        upper="2.00"
+        effort="1.0"
         velocity="0.5"/>
 </joint>
@@ -386,7 +386,7 @@
   <axis xyz="0.0 1.0 0.0"/>
   <!-- Joint limits -->
-  <limit lower="-1.47"
-        upper="1.47"
-        effort="0.5"
+  <limit lower="-2.00"
+        upper="2.00"
+        effort="1.0"
         velocity="0.5"/>
 </joint>
@@ -417,8 +417,8 @@
   <axis xyz="0.0 1.0 0.0"/>
   <!-- Joint limits -->
-  <limit lower="-1.47"
-        upper="1.47"
+  <limit lower="-2.00"
+        upper="2.00"
         effort="1.0"
-        velocity="0.2"/>
+        velocity="0.5"/>
 </joint>
 <joint name="Rigid14" type="fixed">

Commit message: enable global namespace passing for controllers

File: src/edmo_snake_description/urdf/edmo_snake.xacro (robot description, xacro)
@@ -1,4 +1,6 @@
 <?xml version="1.0" ?>
 <robot name="edmo_snake" xmlns:xacro="http://www.ros.org/wiki/xacro">
+<xacro:arg name="robot_prefix" default="" />
+<xacro:property name="robot_prefix" value="$(arg robot_prefix)" />
 <xacro:include filename="$(find edmo_snake_description)/urdf/materials.xacro" />
 <xacro:include filename="$(find edmo_snake_description)/urdf/edmo_snake.trans" />
@@ -437,3 +439,20 @@
   <child link="motor_box_3"/>
 </joint>
+<gazebo>
+  <plugin name="control" filename="libgazebo_ros_control.so">
+    <robotNamespace>${robot_prefix}/edmo_snake_controller</robotNamespace>
+  </plugin>
+</gazebo>
+<gazebo>
+  <plugin name="p3d_base_controller" filename="libgazebo_ros_p3d.so">
+    <alwaysOn>true</alwaysOn>
+    <updateRate>1.0</updateRate>
+    <bodyName>base_link</bodyName>
+    <topicName>${robot_prefix}/edmo_snake/state</topicName>
+    <gaussianNoise>0.0</gaussianNoise>
+    <frameName>world</frameName>
+    <xyzOffsets>0 0 0</xyzOffsets>
+    <rpyOffsets>0 0 0</rpyOffsets>
+  </plugin>
+</gazebo>
 </robot>
